File: kicad6/beagleflash.kicad_pcb (KiCad board)
At the start: 2 copper layers, 86.4 x 54.6 mm, 23 parts, among them P1 SPI-8, P2 SPI-16, P3 EEPROM_PROG_EN, P4 BBB_P9, P5 BBB_P8, P6 CONN_01X01, P7 CONN_01X01, P8 CONN_01X01, P9 CONN_01X01, SW1 DIPS_02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

Commit message: kicad6: Update to kicad version 6
Connections:
- net /~CONN_CS renamed /~{CONN_CS}
- net /~CONN_HOLD renamed /~{CONN_HOLD}
- net /~CONN_WP renamed /~{CONN_WP}
- net /~SPI_CS0 renamed /~{SPI_CS0}
- net /~WP renamed /~{WP}
Other:
- net class Default removed
- net class POWER removed
- board text added: "~{CS}"
- board text added: "~{HOLD}"
- board text added: "~{WP}"
- board text removed: "~CS"
- board text removed: "~HOLD"
- board text removed: "~WP"
