File: kicad6/beagleflash.kicad_sch (KiCad schematic)
At the start: 22 parts

Commit message: kicad6: Fix most of the ERC warnings
Parts:
- C1, C2, C3: value (none) -> 10uF; footprint (none) -> Capacitor_SMD:C_0805_2012Metric
- C4: value (none) -> 0.1uF; footprint (none) -> Capacitor_SMD:C_0805_2012Metric
- H1, H2, H3, H4: value (none) -> M3; footprint (none) -> MountingHole:MountingHole_3.2mm_M3_ISO14580_Pad
- L1: value (none) -> 10uH; footprint (none) -> Inductor_SMD:L_1812_4532Metric
- P1: value (none) -> SPI-8; footprint (none) -> Connector_IDC:IDC-Header_2x05_P2.54mm_Vertical
- P2: value (none) -> SPI-16; footprint (none) -> Connector_IDC:IDC-Header_2x08_P2.54mm_Vertical
- P3: value (none) -> EEPROM_PROG_EN; footprint (none) -> Connector_PinHeader_2.54mm:PinHeader_2x01_P2.54mm_Horizontal
- P4: value (none) -> BBB_P9; footprint (none) -> Connector_PinHeader_2.54mm:PinHeader_2x23_P2.54mm_Vertical
- P5: value (none) -> BBB_P8; footprint (none) -> Connector_PinHeader_2.54mm:PinHeader_2x23_P2.54mm_Vertical
- R1, R2, R3: value (none) -> 10k; footprint (none) -> Resistor_SMD:R_0805_2012Metric
- RP1: value (none) -> 10k; footprint (none) -> Package_SO:SOIC-16_3.9x9.9mm_P1.27mm
- SW1: value (none) -> DIPS_02; footprint (none) -> Button_Switch_THT:SW_DIP_SPSTx02_Slide_9.78x7.26mm_W7.62mm_P2.54mm
- U1: value (none) -> PAM2305AAB330; footprint (none) -> Package_TO_SOT_SMD:TSOT-23-5
- U2: value (none) -> 74HC125; footprint (none) -> Package_SO:SOIC-14_3.9x8.7mm_P1.27mm
- U3: value (none) -> CAT24C256W; footprint (none) -> Package_SO:SOIC-8_3.9x4.9mm_P1.27mm
Connections:
- net SPI_D0: no longer P4.28 (Pin_28), P4.30 (Pin_30), P4.31 (Pin_31), U2.1, U2.10, U2.12, U2.13, U2.2, U2.4, U2.5
- net AGND: no longer names the net of P4.34 (Pin_34)
- net AIN0: no longer names the net of P4.39 (Pin_39)
- net AIN1: no longer names the net of P4.40 (Pin_40)
- net AIN2: no longer names the net of P4.37 (Pin_37)
- net AIN3: no longer names the net of P4.38 (Pin_38)
- net AIN4: no longer names the net of P4.33 (Pin_33)
- net AIN5: no longer names the net of P4.36 (Pin_36)
- net AIN6: no longer names the net of P4.35 (Pin_35)
- net SYS_5V: no longer names the net of P4.7 (Pin_7)
- net SYS_5VB: no longer names the net of P4.8 (Pin_8)
- net VADC: no longer names the net of P4.32 (Pin_32)
- new net SPI_D1: P4.30 (Pin_30), U2.12
- new net SPI_SCLK: P4.31 (Pin_31), U2.5
- new net ~{SPI_CS0}: P4.28 (Pin_28), U2.1, U2.10, U2.13, U2.2, U2.4
